Commit message: changes to make this package specific to NRG

File: motoman_sia5d_support/urdf/sia5d.urdf (robot description, URDF)
Before this commit: robot motoman_sia5d, 10 links, 9 joints
Links:
- added link eef
- added link ft_sensor; collision mesh filename=package://motoman_sia5d_support/meshes/ft_sensor.stl; visual mesh filename=package://motoman_sia5d_support/meshes/ft_sensor.stl
- added link plasma_pen; collision mesh filename=package://motoman_sia5d_support/meshes/pen.stl; visual mesh filename=package://motoman_sia5d_support/meshes/pen.stl
- added link plasma_pen_holder; collision mesh filename=package://motoman_sia5d_support/meshes/plasma_pen_mount.stl; visual mesh filename=package://motoman_sia5d_support/meshes/plasma_pen_mount.stl
- added link tool0_oriented
Joints:
- added joint eef_joint: type fixed, parent plasma_pen, child eef, origin xyz=0.0 0.0 0.23 rpy=0.0 0.0 0.0
- added joint ft_sensor_joint: type fixed, parent tool0_oriented, child ft_sensor, origin xyz=0.0 0.0 0.03 rpy=0.0 0.0 4.15388362029
- added joint ft_to_plasma_joint: type fixed, parent ft_sensor, child plasma_pen_holder, origin xyz=0.0 0.0 0.05 rpy=3.141592654 0.0 4.18879020533
- added joint holder_to_pen: type fixed, parent plasma_pen_holder, child plasma_pen, origin xyz=-0.063 0.0 0.135 rpy=3.141592654 0.0 0.0
- added joint tool0_oriented_joint: type fixed, parent tool0, child tool0_oriented, origin xyz=0.0 0.0 -0.011 rpy=0.0 0.0 0.0

File: motoman_sia5d_support/urdf/sia5d.xacro (robot description, xacro)
@@ -4,3 +4,88 @@
 	<xacro:include filename="$(find motoman_sia5d_support)/urdf/sia5d_macro.xacro"/>
 	<xacro:motoman_sia5d prefix=""/>
+    <!-- properties -->
+    <xacro:property name="M_PI" value="3.141592654" />
+    <xacro:property name="EEF_OFFSET_FROM_ROBOTIQ" value="0.16" />
+    <xacro:property name="FT_OFFSET_FROM_TOOL" value="0.03" />
+    <xacro:property name="FT_ROT" value="238" /> <!-- specify in degrees 238-->
+    <xacro:property name="PLASMA_ROT" value="250" /> <!-- specify in degrees 40 -->
+    <link name="tool0_oriented"></link>
+    <joint name="tool0_oriented_joint" type="fixed">
+      <parent link="tool0" />
+      <child link="tool0_oriented" />
+      <origin xyz="0.0 0.0 -0.011" rpy="0.0 0.0 0.0" />
+    </joint>
+    <!-- attach ft sensor -->
+    <link name="ft_sensor">
+        <visual>
+            <origin rpy="0.0 0.0 0.0" xyz="0.0 0.0 0.0"/>
+            <geometry>
+                <mesh filename="package://motoman_sia5d_support/meshes/ft_sensor.stl"/>
+            </geometry>
+            <material name="silver"/>
+        </visual>
+        <collision>
+            <origin rpy="0 0 0" xyz="0 0 0"/>
+            <geometry>
+                <mesh filename="package://motoman_sia5d_support/meshes/ft_sensor.stl"/>
+            </geometry>
+            <material name="yellow"/>
+        </collision>
+    </link>
+    <joint name="ft_sensor_joint" type="fixed">
+        <parent link="tool0_oriented" />
+        <child link="ft_sensor" />
+        <origin xyz="0.0 0.0 ${FT_OFFSET_FROM_TOOL}" rpy="0.0 0.0 ${FT_ROT*M_PI/180.0}" />
+    </joint>
+    <!-- attach plasma pen holder -->
+    <link name="plasma_pen_holder">
+        <visual>
+            <origin rpy="0 0 0" xyz="0 0 0"/>
+            <geometry>
+                <mesh filename="package://motoman_sia5d_support/meshes/plasma_pen_mount.stl"/>
+            </geometry>
+            <material name="silver"/>
+        </visual>
+        <collision>
+            <origin rpy="0 0 0" xyz="0 0 0"/>
+            <geometry>
+                <mesh filename="package://motoman_sia5d_support/meshes/plasma_pen_mount.stl"/>
+            </geometry>
+            <material name="yellow"/>
+        </collision>
+    </link>
+    <joint name="ft_to_plasma_joint" type="fixed">
+        <parent link="ft_sensor" />
+        <child link="plasma_pen_holder" />
+        <origin xyz="0.0 0.0 0.05" rpy="${180*M_PI/180.0} 0.0 ${240*M_PI/180.0}" />
+    </joint>
+    <!-- attach plasma pen -->
+    <link name="plasma_pen">
+        <visual>
+            <origin rpy="0 0 0" xyz="0 0 0"/>
+            <geometry>
+                <mesh filename="package://motoman_sia5d_support/meshes/pen.stl"/>
+            </geometry>
+            <material name="silver"/>
+        </visual>
+        <collision>
+            <origin rpy="0 0 0" xyz="0 0 0"/>
+            <geometry>
+                <mesh filename="package://motoman_sia5d_support/meshes/pen.stl"/>
+            </geometry>
+            <material name="yellow"/>
+        </collision>
+    </link>
+    <joint name="holder_to_pen" type="fixed">
+        <parent link="plasma_pen_holder" />
+        <child link="plasma_pen" />
+        <origin xyz="-0.063 0.0 0.135" rpy="${180*M_PI/180.0} 0.0 0.0" />
+    </joint>
+    <!-- attach eef link at front of pen -->
+    <link name="eef" />
+    <joint name="eef_joint" type="fixed" >
+        <parent link="plasma_pen" />
+        <child link="eef" />
+        <origin xyz="0.0 0.0 0.23" rpy="0.0 0.0 0.0"/>
+    </joint>
 </robot>

Commit message: changes to make Rviz match SIA5

File: motoman_sia5d_support/urdf/sia5d.urdf (robot description, URDF)
Before this commit: robot motoman_sia5d, 15 links, 14 joints
Links:
- removed link base
Joints:
- removed joint link_l-base
- joint joint_b: axis 0 -1 0 -> 0 1 0; limit lower=-1.91986223 upper=1.91986223 effort=0 velocity=4.01425739 -> lower=-1.919852 upper=1.919852 effort=0 velocity=4.014236
- joint joint_e: limit lower=-2.96705981 upper=2.96705981 effort=0 velocity=3.4906586 -> lower=-2.967044 upper=2.967044 effort=0 velocity=3.49064; origin xyz=0 0 0.27 rpy=0 0 0 -> xyz=0 0 0.27 rpy=0 0 3.141576
- joint joint_l: axis 0 1 0 -> 0 -1 0; limit lower=-1.91986223 upper=1.91986223 effort=0 velocity=3.4906586 -> lower=-1.919852 upper=1.919852 effort=0 velocity=3.49064; origin xyz=0 0 0 rpy=0 0 0 -> xyz=0 0 0 rpy=0 -3.141576 0
- joint joint_r: limit lower=-1.57079637 upper=1.57079637 effort=0 velocity=3.4906586 -> lower=-3.141576 upper=3.141576 effort=0 velocity=3.49064; origin xyz=0.27 0 0.06 rpy=0 0 0 -> xyz=0.27 0 0.060 rpy=0 0 3.141576
- joint joint_s: axis 0 0 1 -> 0 0 -1; limit lower=-3.14159274 upper=3.14159274 effort=0 velocity=3.4906586 -> lower=-3.141576 upper=3.141576 effort=0 velocity=3.49064; origin xyz=0 0 0.31 rpy=0 0 0 -> xyz=0 0 0.31 rpy=3.141576 0 3.141576
- joint joint_t: axis -1 0 0 -> 0 0 1; limit lower=-1.57079637 upper=1.57079637 effort=0 velocity=6.10865255 -> lower=-3.141576 upper=3.141576 effort=0 velocity=6.10862; origin xyz=0.134 0 0 rpy=0 0 0 -> xyz=-0.134 0 0 rpy=0 -1.570788 0
- joint joint_u: limit lower=-1.57079637 upper=2.007128695 effort=0 velocity=3.4906586 -> lower=-1.570788 upper=2.007118 effort=0 velocity=3.49064; origin xyz=0.085 0 0 rpy=0 0 0 -> xyz=-0.085 0 0 rpy=0 0 3.141576
- joint link_t-tool0: origin xyz=0.011 0 0 rpy=-1.57079637 -1.57079637 -1.57079637 -> xyz=0.011 0 0 rpy=-1.570788 -1.570788 -1.570788
- joint tool0_oriented_joint: origin xyz=0.0 0.0 -0.011 rpy=0.0 0.0 0.0 -> xyz=0.0 0.0 -0.011 rpy=0.0 1.570796327 0.0

File: motoman_sia5d_support/urdf/sia5d.xacro (robot description, xacro)
@@ -14,5 +14,5 @@
       <parent link="tool0" />
       <child link="tool0_oriented" />
-      <origin xyz="0.0 0.0 -0.011" rpy="0.0 0.0 0.0" />
+      <origin xyz="0.0 0.0 -0.011" rpy="0.0 ${M_PI/2} 0.0" />
     </joint>
     <!-- attach ft sensor -->

File: motoman_sia5d_support/urdf/sia5d_macro.xacro (robot description, xacro)
@@ -1,5 +1,6 @@
 <?xml version="1.0" ?>
 <robot xmlns:xacro="http://ros.org/wiki/xacro">
-	<xacro:property name="deg" value="0.017453293" /> <!--degrees to radians-->
+	<property name="pi" value="3.141592654" />
+	<property name="deg" value="0.0174532" /> <!--degrees to radians - fudge factor -->
 	<xacro:macro name="motoman_sia5d" params="prefix">
   <link name="${prefix}base_link">
@@ -7,5 +8,5 @@
       <origin xyz="0 0 0" rpy="0 0 0" />
       <geometry>
-        <mesh filename="package://motoman_sia5d_support/meshes/sia5d/visual/base.dae" />
+ 	<mesh filename="package://motoman_sia5d_support/meshes/sia5d/visual/base.dae" />
       </geometry>
     </visual>
@@ -13,5 +14,5 @@
       <origin xyz="0 0 0" rpy="0 0 0" />
       <geometry>
-        <mesh filename="package://motoman_sia5d_support/meshes/sia5d/collision/base.dae" />
+ 	<mesh filename="package://motoman_sia5d_support/meshes/sia5d/collision/base.dae" />
       </geometry>
     </collision>
@@ -19,5 +20,5 @@
   <link name="${prefix}link_s">
     <visual>
-      <origin xyz="0 0 0" rpy="0 0 0" />
+      <origin xyz="0 0 0" rpy="0 ${180*deg} ${180*deg}" />
       <geometry>
         <mesh filename="package://motoman_sia5d_support/meshes/sia5d/visual/link_s.dae" />
@@ -25,5 +26,5 @@
     </visual>
     <collision>
-      <origin xyz="0 0 0" rpy="0 0 0" />
+      <origin xyz="0 0 0" rpy="0 ${180*deg} ${180*deg}" />
       <geometry>
         <mesh filename="package://motoman_sia5d_support/meshes/sia5d/collision/link_s.dae" />
@@ -32,13 +33,13 @@
   </link>
   <joint name="${prefix}joint_s" type="revolute">
-    <origin xyz="0 0 0.31" rpy="0 0 0" /> <!--r=${90*deg}-->
+    <origin xyz="0 0 0.31" rpy="${180*deg} 0 ${180*deg}" />
     <parent link="${prefix}base_link" />
     <child link="${prefix}link_s" />
-    <axis xyz="0 0 1" />
+    <axis xyz="0 0 -1" />
     <limit lower="${-180*deg}" upper="${180*deg}" effort="0" velocity="${200*deg}" />
   </joint>
   <link name="${prefix}link_l">
     <visual>
-      <origin xyz="0 0 0" rpy="0 0 0" />
+      <origin xyz="0 0 0" rpy="0 0 ${-180*deg}" />
       <geometry>
         <mesh filename="package://motoman_sia5d_support/meshes/sia5d/visual/link_l.dae" />
@@ -46,5 +47,5 @@
     </visual>
     <collision>
-      <origin xyz="0 0 0" rpy="0 0 0" />
+      <origin xyz="0 0 0" rpy="0 0 ${-180*deg}" />
       <geometry>
         <mesh filename="package://motoman_sia5d_support/meshes/sia5d/collision/link_l.dae" />
@@ -53,13 +54,13 @@
   </link>
   <joint name="${prefix}joint_l" type="revolute">
-    <origin xyz="0 0 0" rpy="0 0 0" />
+    <origin xyz="0 0 0" rpy="0 ${-180*deg} 0"/>
     <parent link="${prefix}link_s" />
     <child link="${prefix}link_l" />
-    <axis xyz="0 1 0" />
+    <axis xyz="0 -1 0" />
     <limit lower="${-110*deg}" upper="${110*deg}" effort="0" velocity="${200*deg}" />
   </joint>
   <link name="${prefix}link_e">
     <visual>
-      <origin xyz="0 0 0" rpy="0 0 0" />
+      <origin xyz="0 0 0" rpy="0 0 ${180*deg}" />
       <geometry>
         <mesh filename="package://motoman_sia5d_support/meshes/sia5d/visual/link_e.dae" />
@@ -67,5 +68,5 @@
     </visual>
     <collision>
-      <origin xyz="0 0 0" rpy="0 0 0" />
+      <origin xyz="0 0 0" rpy="0 0 ${180*deg}" />
       <geometry>
         <mesh filename="package://motoman_sia5d_support/meshes/sia5d/collision/link_e.dae" />
@@ -74,5 +75,5 @@
   </link>
   <joint name="${prefix}joint_e" type="revolute">
-    <origin xyz="0 0 0.27" rpy="0 0 0" />
+    <origin xyz="0 0 0.27" rpy="0 0 ${180*deg}"/>
     <parent link="${prefix}link_l" />
     <child link="${prefix}link_e" />
@@ -95,5 +96,5 @@
   </link>
   <joint name="${prefix}joint_u" type="revolute">
-    <origin xyz="0.085 0 0" rpy="0 0 0" />
+    <origin xyz="-0.085 0 0" rpy="0 0 ${180*deg}"/>
     <parent link="${prefix}link_e" />
     <child link="${prefix}link_u" />
@@ -103,5 +104,5 @@
   <link name="${prefix}link_r">
     <visual>
-      <origin xyz="0 0 0" rpy="0 0 0" />
+      <origin xyz="0 0 0" rpy="0 0 ${180*deg}" />
       <geometry>
         <mesh filename="package://motoman_sia5d_support/meshes/sia5d/visual/link_r.dae" />
@@ -109,5 +110,5 @@
     </visual>
     <collision>
-      <origin xyz="0 0 0" rpy="0 0 0" />
+      <origin xyz="0 0 0" rpy="0 0 ${180*deg}" />
       <geometry>
         <mesh filename="package://motoman_sia5d_support/meshes/sia5d/collision/link_r.dae" />
@@ -116,13 +117,13 @@
   </link>
   <joint name="${prefix}joint_r" type="revolute">
-    <origin xyz="0.27 0 0.06" rpy="0 0 0" />
+    <origin xyz="0.27 0 0.060" rpy="0 0 ${180*deg}"/>
     <parent link="${prefix}link_u" />
     <child link="${prefix}link_r" />
     <axis xyz="-1 0 0" />
-    <limit lower="${-90*deg}" upper="${90*deg}" effort="0" velocity="${200*deg}" />
+    <limit lower="${-180*deg}" upper="${180*deg}" effort="0" velocity="${200*deg}" />
   </joint>
   <link name="${prefix}link_b">
     <visual>
-      <origin xyz="0 0 0" rpy="0 0 0" />
+      <origin xyz="0 0 0" rpy="0 0 ${180*deg}" />
       <geometry>
         <mesh filename="package://motoman_sia5d_support/meshes/sia5d/visual/link_b.dae" />
@@ -130,5 +131,5 @@
     </visual>
     <collision>
-      <origin xyz="0 0 0" rpy="0 0 0" />
+      <origin xyz="0 0 0" rpy="0 0 ${180*deg}" />
       <geometry>
         <mesh filename="package://motoman_sia5d_support/meshes/sia5d/collision/link_b.dae" />
@@ -140,10 +141,10 @@
     <parent link="${prefix}link_r" />
     <child link="${prefix}link_b" />
-    <axis xyz="0 -1 0" />
+    <axis xyz="0 1 0" />
     <limit lower="${-110*deg}" upper="${110*deg}" effort="0" velocity="${230*deg}" />
   </joint>
   <link name="${prefix}link_t">
     <visual>
-      <origin xyz="0 0 0" rpy="0 0 0" />
+      <origin xyz="0 0 0" rpy="0 ${-90*deg} 0" />
       <geometry>
         <mesh filename="package://motoman_sia5d_support/meshes/sia5d/visual/link_t.dae" />
@@ -151,5 +152,5 @@
     </visual>
     <collision>
-      <origin xyz="0 0 0" rpy="0 0 0" />
+      <origin xyz="0 0 0" rpy="0 ${-90*deg} 0" />
       <geometry>
         <mesh filename="package://motoman_sia5d_support/meshes/sia5d/collision/link_t.dae" />
@@ -158,9 +159,9 @@
   </link>
   <joint name="${prefix}joint_t" type="revolute">
-    <origin xyz="0.134 0 0" rpy="0 0 0" />
+    <origin xyz="-0.134 0 0" rpy="0 ${-90*deg} 0"/>
     <parent link="${prefix}link_b" />
     <child link="${prefix}link_t" />
-    <axis xyz="-1 0 0" />
-    <limit lower="${-90*deg}" upper="${90*deg}" effort="0" velocity="${350*deg}" />
+    <axis xyz="0 0 1" />
+    <limit lower="${-180*deg}" upper="${180*deg}" effort="0" velocity="${350*deg}" />
   </joint>
   <link name="${prefix}tool0" />
@@ -170,11 +171,4 @@
     <child link="${prefix}tool0" />
   </joint>
-    <!-- ROS base_link (via link_l) to Motoman Robot (not Base) Frame transform -->
-    <link name="${prefix}base" />
-    <joint name="${prefix}link_l-base" type="fixed">
-      <origin xyz="0 0 0" rpy="0 0 0"/>
-      <parent link="${prefix}link_l"/>
-      <child link="${prefix}base"/>
-    </joint>
 	</xacro:macro>
 </robot>
